File: Shield/PCB/Shield-Proteco.sch (EAGLE design)
At the start: 28 parts

Commit message: Avance shield y correccion librerias
Parts:
- removed M-LEFT, M-RIGHT: POLOLU-MICROMOTOR, Motores:POLOLU-MICROMOTOR
- added ARDUINO-MEGA: ARDUINO_MEGA, Arduino:ARDUINO_MEGA
- added LED1, LED2, LED3, LED4, LED5: (no value), led:LEDCHIPLED_1206
- added R10, R11, R12, R13, R14: (no value), rcl:R-US_M1206
- added U$14: TFT_ARDUINO-UNO-MEGA, TFT:TFT_ARDUINO-UNO-MEGA
- added U$15: ACELEROMETER-MPU6050-JST, Sensores:ACELEROMETER-MPU6050-JST
- added U$16, U$17: SERVOMOTORES, Motores:SERVOMOTORES
- added U$18: SLIDE-3, Interruptores:SLIDE-3
- added U$3, U$6: TB6612FNG, Driver-Motor:TB6612FNG
- added U$7, U$8: POLOLU-MICROMOTOR, Motores:POLOLU-MICROMOTOR
- U$1: value ARDUINO_MEGA -> SERVOMOTORES; device Arduino:ARDUINO_MEGA -> Motores:SERVOMOTORES
- renumbered BT-PROG to U$13, LINE-SENSOR to U$12, SHARP-LEFT to U$9, SHARP-MIDD to U$10, SHARP-RIGHT to U$11
Connections:
- new net N$17: U$15.SCL
- new net N$18: U$15.SDA
- new net N$19: U$15.XDA
- new net N$20: U$15.XCL
- new net N$21: U$15.ADO
- new net N$22: U$15.INT
- new net N$23: LED1.C, R10.2
- new net N$24: LED2.C, R11.2
- new net N$25: LED3.C, R12.2
- new net N$26: LED4.C, R13.2
- new net N$27: U$14.NC_5
- new net N$28: U$14.3V3
- new net N$29: U$14.5V, U$18.P2
- new net N$30: U$14.NC_3
- new net N$31: U$14.GND
- new net N$32: U$14.NC_2
- new net N$33: U$14.LCD_RD
- new net N$34: U$14.LCD_WR
- new net N$35: U$14.LCD_RS
- new net N$36: U$14.LCD_CS
- new net N$37: U$14.LCD_RST
- new net N$38: U$14.NC_1
- new net N$39: ARDUINO-MEGA.3V3
- new net N$40: ARDUINO-MEGA.5V_1
- new net N$41: ARDUINO-MEGA.GND_2
- new net N$42: ARDUINO-MEGA.GND_1
- new net N$43: ARDUINO-MEGA.VIN
- new net N$44: ARDUINO-MEGA.A0
- new net N$45: ARDUINO-MEGA.A1
- new net N$46: ARDUINO-MEGA.A2
- new net N$47: ARDUINO-MEGA.A3
- new net N$48: ARDUINO-MEGA.A4
- new net N$49: ARDUINO-MEGA.A5
- new net N$50: ARDUINO-MEGA.A6
- new net N$51: ARDUINO-MEGA.A7
- new net N$52: ARDUINO-MEGA.A8
- new net N$53: ARDUINO-MEGA.A9
- new net N$54: ARDUINO-MEGA.A10
- new net N$55: ARDUINO-MEGA.A11
- new net N$56: ARDUINO-MEGA.A12
- new net N$57: ARDUINO-MEGA.A13
- new net N$58: ARDUINO-MEGA.A14
- new net N$59: ARDUINO-MEGA.A15
- new net N$60: U$14.NC_6
- new net N$61: U$14.LCD_D2
- new net N$62: U$14.LCD_D3
- new net N$63: U$14.LCD_D4
- new net N$64: U$14.LCD_D5
- new net N$65: U$14.LCD_D6
- new net N$66: U$14.LCD_D7
- new net N$67: U$14.NC_8
- new net N$68: U$14.NC_7
- new net N$70: U$14.SD_DO
- new net N$71: U$14.SD_DI
- new net N$72: U$14.SD_SS
- new net N$73: U$14.LCD_D1
- new net N$74: U$14.LCD_D0
- new net N$75: U$1.SIGNAL
- new net N$76: U$16.SIGNAL
- new net N$77: U$17.SIGNAL
- new net N$78: ARDUINO-MEGA.SCL
- new net N$79: ARDUINO-MEGA.SDA
- new net N$80: ARDUINO-MEGA.AREF
- new net N$81: ARDUINO-MEGA.GND
- new net SD_SCK: ARDUINO-MEGA.13, U$14.SD_SCK
- net 6V-DC-3A: now also U$3.VM, U$6.VM; no longer M-LEFT.VCC, M-RIGHT.VCC
- net GND: now also R10.1, R11.1, R12.1, R13.1, R14.1, U$1.GND, U$15.GND, U$16.GND, U$17.GND, U$3.GND, U$3.GND_1, U$3.GND_2, U$6.GND, U$6.GND_1, U$6.GND_2, U$7.GND, U$8.GND; no longer M-LEFT.GND, M-RIGHT.GND
- net RESET: now also ARDUINO-MEGA.RESET, U$14.NC_4
- net VCC: now also U$1.VCC, U$15.VCC, U$16.VCC, U$17.VCC, U$18.COM, U$3.VCC, U$6.VCC, U$7.VCC, U$8.VCC

Commit message: Avance Shield
Parts:
- added D1, D2: (no value), zetex:DSOD323
- added LED6: (no value), led:LEDCHIPLED_1206
- added R15: (no value), rcl:R-US_M1206
- added SHARP-LEFT, SHARP-MIDDLE: SHARP, Sensores:SHARP
- U$10: value SHARP -> SERVOMOTORES; device Sensores:SHARP -> Motores:SERVOMOTORES
- U$9: value SHARP -> SENSOR-MISCELANEOUS; device Sensores:SHARP -> Sensores:SENSOR-MISCELANEOUS
- renumbered SG1 to BUZZER, T1 to BC547, U$11 to SHARP-RIGHT, U$13 to HC-05
Connections:
- new net LED1: LED1.A
- new net LED2: LED2.A
- new net LED3: LED3.A
- new net LED4: LED4.A
- new net LED5: LED5.A
- new net N$100: U$3.AO2, U$3.BO2
- new net N$101: U$3.AO1, U$3.BO1
- new net N$102: U$7.OUTB
- new net N$103: U$7.OUTA
- new net N$104: U$7.M2
- new net N$105: U$7.M1
- new net N$106: U$8.OUTA
- new net N$107: U$8.OUTB
- new net N$108: U$8.M2
- new net N$109: U$8.M1
- new net N$110: U$9.3.3V
- new net N$111: ARDUINO-MEGA.12
- new net N$112: ARDUINO-MEGA.11
- new net N$113: ARDUINO-MEGA.10
- new net N$114: ARDUINO-MEGA.9
- new net N$115: ARDUINO-MEGA.8
- new net N$116: ARDUINO-MEGA.7
- new net N$117: ARDUINO-MEGA.6
- new net N$69: U$9.E1
- new net N$82: U$9.E2
- new net N$83: U$9.E3
- new net N$84: U$9.E4
- new net N$85: U$9.E5
- new net N$86: U$9.E6
- new net N$87: U$9.E7
- new net N$88: LED5.C, R14.2
- new net N$89: LED6.C, R15.2
- new net N$90: D2.A, HC-05.TX
- new net N$91: D1.C, HC-05.RX
- new net N$92: U$6.AIN1, U$6.BIN1
- new net N$93: U$6.AIN2, U$6.BIN2
- new net N$94: U$6.AO2, U$6.BO2
- new net N$95: U$6.AO1, U$6.BO1
- new net N$96: U$6.PWMA, U$6.PWMB
- new net N$97: U$3.AIN1, U$3.BIN1
- new net N$98: U$3.AIN2, U$3.BIN2
- new net N$99: U$3.PWMA, U$3.PWMB
- net GND: now also R15.1, SHARP-LEFT.GND, SHARP-MIDDLE.GND
- net N$10: now also S2.P1
- net N$11: now also S1.P1
- net N$12: now also S3.P1
- net N$13: now also S4.P1
- net N$7: now also SHARP-LEFT.DISTANCE; no longer U$9.DISTANCE
- net N$77: now also U$10.SIGNAL
- net N$8: now also SHARP-MIDDLE.DISTANCE; no longer U$10.DISTANCE
- net RX0: now also D2.C; no longer HC-05.RX
- net TX0: now also D1.A; no longer HC-05.TX
- net VCC: now also LED6.A, SHARP-LEFT.VCC, SHARP-MIDDLE.VCC
Other:
- moved on the sheet: R1, R2, R3, R4, SW2, U$18
