File: Shield/BT-PROGRAMER/BT-PROGRAMER.brd (EAGLE design)
At the start: 18 x 27.2 mm, 10 parts

Commit message: Más avance
Routing:
- added copper zone on layer 1, net GND
Changed lines of the file:
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@@
 <wire x1="16.688" y1="26.66" x2="-1.27" y2="26.66" width="0" layer="20"/>
 <wire x1="-1.27" y1="26.66" x2="-1.27" y2="-0.508" width="0" layer="20"/>
-<dimension x1="-1.27" y1="-0.508" x2="16.688" y2="-0.508" x3="7.709" y3="-3.048" textsize="1.778" layer="1"/>
-<dimension x1="16.688" y1="-0.508" x2="16.688" y2="26.66" x3="20.828" y3="13.076" textsize="1.778" layer="1"/>
 </plain>
 <attributes>
@@
 <wire x1="1.785" y1="14.478" x2="2.293" y2="14.478" width="0.3048" layer="1"/>
 <wire x1="2.54" y1="11.56" x2="3.048" y2="12.068" width="0.3048" layer="1"/>
+<polygon width="0.1524" layer="1" isolate="0.4064">
+<vertex x="-1.27" y="25.654"/>
+<vertex x="-1.27" y="25.908"/>
+<vertex x="-0.508" y="26.67"/>
+<vertex x="15.748" y="26.67"/>
+<vertex x="16.764" y="25.654"/>
+<vertex x="16.764" y="0.508"/>
+<vertex x="15.748" y="-0.508"/>
+<vertex x="-0.254" y="-0.508"/>
+<vertex x="-1.27" y="0.508"/>
+</polygon>
 </signal>
 <signal name="VCC">
