File: Shield/BT-PROGRAMER/BT-PROGRAMER.brd (EAGLE design)
At the start: 18 x 27.2 mm, 10 parts

Commit message: Shield Terminada
Routing:
- net VCC: vias 0 -> 1
- net N$2: vias 0 -> 1
- net GND: vias 0 -> 1
