File: Shield/Shield-Proteco.sch (EAGLE design)
At the start: 52 parts, among them Q1 FDD4141TO252

Commit message: Preruteo
Parts:
- added LED5: (no value), led:LEDCHIPLED_1206
- added PUSH3, PUSH4: (no value), switch-omron:10-XX
- added R-PUSH3, RLED-5, RPUSH-4: (no value), rcl:R-US_M1206
- renumbered PUSH to PUSH2
Connections:
- removed net ENC1-LEFT: ARDUINO-MEGA.14-TX3, MOTOR_LEFT.M1
- removed net ENC1-RIGHT: ARDUINO-MEGA.18-TX1, MOTOR_RIGHT.M1
- removed net ENC2-LEFT: ARDUINO-MEGA.15-RX3, MOTOR_LEFT.M2
- removed net ENC2-RIGHT: ARDUINO-MEGA.A8, MOTOR_RIGHT.M2
- removed net LED1W: ARDUINO-MEGA.45
- removed net N$1: U$9.E8
- removed net N$10: ARDUINO-MEGA.49
- removed net N$11: ARDUINO-MEGA.51
- removed net N$12: ARDUINO-MEGA.53
- removed net N$28: ARDUINO-MEGA.30
- removed net N$29: ARDUINO-MEGA.34
- removed net N$30: ARDUINO-MEGA.38
- removed net N$31: ARDUINO-MEGA.42
- removed net N$32: ARDUINO-MEGA.46
- removed net N$33: ARDUINO-MEGA.50
- removed net N$36: ARDUINO-MEGA.28
- removed net N$37: ARDUINO-MEGA.32
- removed net N$39: ARDUINO-MEGA.36
- removed net N$40: ARDUINO-MEGA.40
- removed net N$41: ARDUINO-MEGA.44
- removed net N$42: ARDUINO-MEGA.48
- removed net N$43: ARDUINO-MEGA.52
- removed net PUSH: ARDUINO-MEGA.25, PUSH2.P, PUSH2.P1, RPUSH-2.2
- new net ENC-LEFT1: ARDUINO-MEGA.18-TX1, MOTOR_LEFT.M1
- new net ENC-LEFT2: ARDUINO-MEGA.19-RX1, MOTOR_LEFT.M2
- new net ENC-RIGHT1: ARDUINO-MEGA.20-SDA, MOTOR_RIGHT.M1
- new net ENC-RIGHT2: ARDUINO-MEGA.21-SCL, MOTOR_RIGHT.M2
- new net LED5: LED5.A
- new net N$119: ARDUINO-MEGA.14-TX3
- new net N$120: ARDUINO-MEGA.15-RX3
- new net N$49: ARDUINO-MEGA.A5
- new net N$50: ARDUINO-MEGA.A6
- new net N$51: ARDUINO-MEGA.A7
- new net N$52: ARDUINO-MEGA.A8
- new net N$88: LED5.C, RLED-5.2
- new net PUSH2: PUSH2.P, PUSH2.P1, RPUSH-2.2
- new net PUSH3: PUSH3.P, PUSH3.P1, R-PUSH3.2
- new net PUSH4: PUSH4.P, PUSH4.P1, RPUSH-4.2
- net BUZZER: no longer ARDUINO-MEGA.35
- net DIP1: no longer ARDUINO-MEGA.23
- net DIP2: no longer ARDUINO-MEGA.22, ARDUINO-MEGA.5V_3
- net DIP3: no longer ARDUINO-MEGA.24
- net DIP4: no longer ARDUINO-MEGA.26
- net GND: now also R-PUSH3.1, RLED-5.1, RPUSH-4.1
- net INT: no longer ARDUINO-MEGA.19-RX1
- net LED1: no longer ARDUINO-MEGA.27
- net LED2: no longer ARDUINO-MEGA.29
- net LED3: no longer ARDUINO-MEGA.31
- net LED4: no longer ARDUINO-MEGA.33
- net SCI: no longer ARDUINO-MEGA.47
- net SCL: no longer ARDUINO-MEGA.21-SCL
- net SDA: no longer ARDUINO-MEGA.20-SDA
- net SERVO1: no longer ARDUINO-MEGA.37
- net SERVO2: no longer ARDUINO-MEGA.39
- net SERVO3: no longer ARDUINO-MEGA.41
- net SERVO4: no longer ARDUINO-MEGA.43
- net SHARP-LEFT: no longer ARDUINO-MEGA.A5
- net SHARP-MIDDLE: no longer ARDUINO-MEGA.A6
- net SHARP-RIGHT: no longer ARDUINO-MEGA.A7
- net VCC: now also PUSH3.S, PUSH4.S
