File: Shield/Shield/Shield-Proteco.brd (EAGLE design)
At the start: 98.7 x 81.3 mm, 52 parts, among them Q1 FDD4141TO252

Commit message: Conexiones
Parts:
- removed PUSH2: (no value), switch-omron:B3F-10XX
- added PUSH: (no value), switch-omron:B3F-10XX
- moved SERVO_1 91.2 mm to (92.1, 36.8), turned to 270 degrees
- moved DS1 83.2 mm to (84.5, 38.7)
- moved SERVO_2 79.0 mm to (92.1, 26.7), turned to 270 degrees
- moved SERVO_3 67.5 mm to (92.1, 16.5), turned to 270 degrees
- moved SERVO_4 51.7 mm to (85.7, 21.0), turned to 270 degrees
- moved DS2 31.5 mm to (84.5, 35.6), turned to 0 degrees
- moved RLED-PWR 27.6 mm to (91.4, 56.5), turned to 180 degrees
- moved DS3 27.5 mm to (84.5, 32.4), turned to 0 degrees
- moved LED-PWR 24.0 mm to (85.7, 55.2), turned to 270 degrees
- moved DS4 22.9 mm to (84.5, 28.6), turned to 0 degrees
- moved MOTOR_RIGHT 22.3 mm to (29.2, 10.2)
- moved RLED-1 21.5 mm to (91.4, 53.3), turned to 180 degrees
- moved LED1 19.1 mm to (85.7, 52.7), turned to 270 degrees
- moved MOTOR_LEFT 18.2 mm to (10.8, 10.2)
- moved RLED-2 15.6 mm to (91.4, 50.2), turned to 180 degrees
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Connections:
- removed net N$1: U$9.E8
- removed net N$104: MOTOR_LEFT.M2
- removed net N$105: MOTOR_LEFT.M1
- removed net N$108: MOTOR_RIGHT.M2
- removed net N$109: MOTOR_RIGHT.M1
- removed net N$119: ARDUINO-MEGA.14-TX3
- removed net N$120: ARDUINO-MEGA.15-RX3
- removed net N$121: ARDUINO-MEGA.16-TX2
- removed net N$122: ARDUINO-MEGA.17-RX2
- removed net N$123: ARDUINO-MEGA.18-TX1
- removed net N$124: ARDUINO-MEGA.19-RX1
- removed net N$125: ARDUINO-MEGA.20
- removed net N$126: ARDUINO-MEGA.21
- removed net N$129: U$9.E9
- removed net N$130: U$9.E10
- removed net N$131: U$9.E11
- removed net N$132: U$9.E12
- removed net N$133: U$9.E13
- removed net N$49: ARDUINO-MEGA.A5
- removed net N$50: ARDUINO-MEGA.A6
- removed net N$51: ARDUINO-MEGA.A7
- removed net N$52: ARDUINO-MEGA.A8
- removed net N$53: ARDUINO-MEGA.A9
- removed net N$54: ARDUINO-MEGA.A10
- removed net N$55: ARDUINO-MEGA.A11
- removed net N$56: ARDUINO-MEGA.A12
- removed net N$57: ARDUINO-MEGA.A13
- removed net N$58: ARDUINO-MEGA.A14
- removed net N$59: ARDUINO-MEGA.A15
- removed net N$69: U$9.E1
- removed net N$82: U$9.E2
- removed net N$83: U$9.E3
- removed net N$84: U$9.E4
- removed net N$85: U$9.E5
- removed net N$86: U$9.E6
- removed net N$87: U$9.E7
- removed net PUSH2: PUSH2.3, PUSH2.4, RPUSH-2.2
- new net A10: ARDUINO-MEGA.A10, U$9.E4
- new net A11: ARDUINO-MEGA.A11, U$9.E5
- new net A12: ARDUINO-MEGA.A12, U$9.E6
- new net A13: ARDUINO-MEGA.A13, U$9.E7
- new net A14: ARDUINO-MEGA.A14, U$9.E8
- new net A15: ARDUINO-MEGA.A15, U$9.E9
- new net A9: ARDUINO-MEGA.A9, U$9.E3
- new net D36: ARDUINO-MEGA.36, U$9.E10
- new net D38: ARDUINO-MEGA.38, U$9.E11
- new net D40: ARDUINO-MEGA.40, U$9.E12
- new net D42: ARDUINO-MEGA.42, U$9.E13
- new net ENC1-LEFT: ARDUINO-MEGA.14-TX3, MOTOR_LEFT.M1
- new net ENC1-RIGHT: ARDUINO-MEGA.18-TX1, MOTOR_RIGHT.M1
- new net ENC2-LEFT: ARDUINO-MEGA.15-RX3, MOTOR_LEFT.M2
- new net ENC2-RIGHT: ARDUINO-MEGA.A8, MOTOR_RIGHT.M2
- new net LED1W: ARDUINO-MEGA.45
- new net N$10: ARDUINO-MEGA.49
- new net N$11: ARDUINO-MEGA.51
- new net N$12: ARDUINO-MEGA.53
- new net N$33: ARDUINO-MEGA.50
- new net N$42: ARDUINO-MEGA.48
- new net N$43: ARDUINO-MEGA.52
- new net PUSH: ARDUINO-MEGA.25, PUSH.3, PUSH.4, RPUSH-2.2
- new net RX2: ARDUINO-MEGA.17-RX2, U$9.E1
- new net TX2: ARDUINO-MEGA.16-TX2, U$9.E2
- net BUZZER: now also ARDUINO-MEGA.35
- net DIP1: now also ARDUINO-MEGA.23
- net DIP2: now also ARDUINO-MEGA.22, ARDUINO-MEGA.5V_3
- net DIP3: now also ARDUINO-MEGA.24
- net DIP4: now also ARDUINO-MEGA.26
- net INT: now also ARDUINO-MEGA.19-RX1
- net LED1: now also ARDUINO-MEGA.27
- net LED2: now also ARDUINO-MEGA.29
- net LED3: now also ARDUINO-MEGA.31
- net LED4: now also ARDUINO-MEGA.33
- net OUT1-MOTOR-LEFT: now also ARDUINO-MEGA.28
- net OUT1-MOTOR-RIGHT: now also ARDUINO-MEGA.32
- net OUT2-MOTOR-LEFT: now also ARDUINO-MEGA.30
- net OUT2-MOTOR-RIGHT: now also ARDUINO-MEGA.34
- net PWM-MOTOR-LEFT: now also ARDUINO-MEGA.44
- net PWM-MOTOR-RIGHT: now also ARDUINO-MEGA.46
- net SCI: now also ARDUINO-MEGA.47
- net SCL: now also ARDUINO-MEGA.21
- net SDA: now also ARDUINO-MEGA.20
- net SERVO1: now also ARDUINO-MEGA.37
- net SERVO2: now also ARDUINO-MEGA.39
- net SERVO3: now also ARDUINO-MEGA.41
- net SERVO4: now also ARDUINO-MEGA.43
- net SHARP-LEFT: now also ARDUINO-MEGA.A5
- net SHARP-MIDDLE: now also ARDUINO-MEGA.A6
- net SHARP-RIGHT: now also ARDUINO-MEGA.A7
- net VCC: now also PUSH.1; no longer PUSH2.1

Commit message: Preruteo
Parts:
- removed Q1: FDD4141TO252, transistor-fet:TO252
- added Q2: TIP41C, transistor-power:TO220AV
- added R-LP: (no value), rcl:M1206
- moved BC547 51.7 mm to (94.6, 62.2), turned to 180 degrees
- moved BUZZER 50.8 mm to (93.3, 74.3), turned to 180 degrees
- moved SW_FAN1 49.4 mm to (90.8, 26.7)
- moved LED_1W 48.8 mm to (95.9, 29.2), turned to 180 degrees
- moved SW_FAN_AUX 42.5 mm to (90.8, 21.6), turned to 180 degrees
- moved FAN1 41.6 mm to (95.9, 16.5)
- moved U$9 38.7 mm to (62.2, 39.4), turned to 270 degrees
- moved PUSH-RST 38.1 mm to (47.6, 71.8), turned to 180 degrees
- moved FAN_AUX 31.5 mm to (90.8, 16.5)
- moved R_BUZZ 30.7 mm to (84.5, 52.1), turned to 0 degrees
- moved SERVO_3 29.9 mm to (94.0, 46.4), turned to 0 degrees
- moved SERVO_2 24.8 mm to (94.0, 51.4), turned to 0 degrees
- moved RLED-4 23.5 mm to (92.7, 67.3), turned to 270 degrees
- moved LINE-SENSOR 22.9 mm to (85.7, 19.1)
- moved LED-PWR 22.2 mm to (85.1, 77.5), turned to 180 degrees
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Connections:
- removed net DRAIN: Q1.3
- removed net GATE: Q1.1
- removed net N$10: ARDUINO-MEGA.49
- removed net N$11: ARDUINO-MEGA.51
- removed net N$12: ARDUINO-MEGA.53
- removed net N$33: ARDUINO-MEGA.50
- removed net N$42: ARDUINO-MEGA.48
- removed net N$43: ARDUINO-MEGA.52
- removed net SOURCE: Q1.2
- new net IOREF: ARDUINO-MEGA.IOREF, U$14.IOREF
- new net N$1: LED_1W.2, Q2.C
- new net N$2: Q2.B, R-LP.2
- new net NC: ARDUINO-MEGA.NC, U$14.NC
- net A10: now also U$9.E7; no longer U$9.E4
- net A11: now also U$9.E9; no longer U$9.E5
- net A12: now also U$9.E11; no longer U$9.E6
- net A13: now also U$9.E13; no longer U$9.E7
- net A14: now also U$9.E12; no longer U$9.E8
- net A15: now also U$9.E10; no longer U$9.E9
- net A9: now also U$9.E5; no longer U$9.E3
- net D36: now also U$9.E2; no longer U$9.E10
- net D38: now also U$9.E4; no longer U$9.E11
- net D40: now also U$9.E6; no longer U$9.E12
- net D42: now also U$9.E8; no longer U$9.E13
- net DIP2: no longer ARDUINO-MEGA.5V_3
- net GND: now also Q2.E
- net LED1W: now also R-LP.1
- net SCD: now also ARDUINO-MEGA.50
- net SF: now also ARDUINO-MEGA.48
- net SID: now also ARDUINO-MEGA.53
- net SII: now also ARDUINO-MEGA.51
- net SSD: now also ARDUINO-MEGA.52
- net SSI: now also ARDUINO-MEGA.49
- net TX2: now also U$9.E3; no longer U$9.E2
- net VCC: now also LED_1W.1
Other:
- board size 98.7 x 81.3 mm -> 110.2 x 79.4 mm
