File: Shield/Shield/Shield-Proteco.brd (EAGLE design)
At the start: 110.2 x 79.4 mm, 53 parts, among them Q2 TIP41C

Commit message: Ruteo
Parts:
- moved U$9 4.12 mm to (65.7, 41.7)
- moved BUZZER 3.82 mm to (96.9, 75.7), turned to 270 degrees
- moved RPUSH-2 3.29 mm to (83.4, 74.5), turned to 180 degrees
- moved SERVO_1 2.85 mm to (96.4, 55.0)
- moved SERVO_2 2.85 mm to (96.4, 49.9)
- moved SERVO_4 2.85 mm to (96.4, 39.8)
- moved SERVO_3 2.85 mm to (96.4, 44.8)
- moved BC547 1.82 mm to (96.4, 61.8)
- moved LED-PWR 1.80 mm to (83.3, 77.2), turned to 270 degrees
- moved PUSH 1.09 mm to (75.3, 74.3)
- moved RLED-PWR 0.97 mm to (83.4, 71.5)
- moved R-DIP4 0.92 mm to (70.1, 59.3)
- moved R-DIP1 0.85 mm to (60.7, 59.2)
- moved R-DIP3 0.80 mm to (66.9, 59.2)
- moved RLED-1 0.80 mm to (82.4, 67.1)
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Connections:
- removed net N$38: U$14.A5
- net GND: no longer 5V-SOURCE.OUT-, MOTORS-SOURCE.OUT-
- net PUSH: no longer PUSH.4
- net RESET: no longer PUSH-RST.3
- net SCL: no longer ARDUINO-MEGA.SCL
- net SDA: no longer ARDUINO-MEGA.SDA
- net SHARP-LEFT: now also U$14.A5
Routing:
- net GND: track 0.00 -> 366.1 mm, vias 0 -> 1
- net VCC: track 0.00 -> 259.2 mm
- net N$14: track 0.00 -> 76.5 mm
- net PWM-MOTOR-LEFT: track 0.00 -> 65.0 mm
- net PWM-MOTOR-RIGHT: track 0.00 -> 60.9 mm
- net OUT1-MOTOR-LEFT: track 0.00 -> 55.7 mm
- net 6V-DC-3A: track 0.00 -> 51.1 mm
- net OUT2-MOTOR-LEFT: track 0.00 -> 48.8 mm
- net OUT1-MOTOR-RIGHT: track 0.00 -> 30.6 mm
- net A9: track 0.00 -> 30.4 mm
- net SF: track 0.00 -> 30.0 mm, vias 0 -> 1
- net INT: track 0.00 -> 28.7 mm
- net SCL: track 0.00 -> 28.3 mm
- net SDA: track 0.00 -> 28.2 mm
- net RX0: track 0.00 -> 27.0 mm
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Other:
- board size 110.2 x 79.4 mm -> 114.7 x 79.5 mm

Commit message: Ruteo avance
Parts:
- moved BUZZER 3.37 mm to (93.7, 76.8)
- moved MOTOR_LEFT 0.63 mm to (10.8, 9.53)
- moved MOTOR_RIGHT 0.63 mm to (29.2, 9.53)
Connections:
- net IN1-MOTOR-LEFT: now also ARDUINO-MEGA.30
- net IN1-MOTOR-RIGHT: now also ARDUINO-MEGA.32
- net IN2-MOTOR-LEFT: now also ARDUINO-MEGA.28
- net IN2-MOTOR-RIGHT: now also ARDUINO-MEGA.34
- net OUT1-MOTOR-LEFT: no longer ARDUINO-MEGA.28
- net OUT1-MOTOR-RIGHT: no longer ARDUINO-MEGA.32
- net OUT2-MOTOR-LEFT: no longer ARDUINO-MEGA.30
- net OUT2-MOTOR-RIGHT: no longer ARDUINO-MEGA.34
Routing:
- net VCC: track 259.2 -> 403.9 mm, vias 0 -> 1
- net GND: track 366.1 -> 479.0 mm, vias 1 -> 3
- net ENC1-LEFT: track 0.00 -> 108.2 mm, vias 0 -> 2
- net ENC2-LEFT: track 0.00 -> 105.5 mm, vias 0 -> 2
- net ENC1-RIGHT: track 0.00 -> 87.2 mm, vias 0 -> 2
- net RESET: track 12.5 -> 94.8 mm, vias 0 -> 1
- net IN2-MOTOR-RIGHT: track 9.01 -> 72.4 mm, vias 0 -> 3
- net IN1-MOTOR-RIGHT: track 15.7 -> 78.2 mm, vias 0 -> 3
- net IN1-MOTOR-LEFT: track 7.77 -> 65.8 mm, vias 0 -> 1
- net IN2-MOTOR-LEFT: track 15.2 -> 62.7 mm, vias 0 -> 1
- net OUT2-MOTOR-RIGHT: track 24.0 -> 70.9 mm, vias 0 -> 2
- net 3V3: track 0.00 -> 44.4 mm, vias 0 -> 1
- net OUT1-MOTOR-RIGHT: track 30.6 -> 73.7 mm, vias 0 -> 2
- net ENC2-RIGHT: track 0.00 -> 30.5 mm, vias 0 -> 2
- net OUT1-MOTOR-LEFT: track 55.7 -> 83.2 mm, vias 0 -> 2
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
Commit message: More Route
Parts:
- moved PUSH 1.20 mm to (75.9, 75.3)
Routing:
- net DIP1: track 12.5 -> 48.8 mm
- net 3V3: track 44.4 -> 77.4 mm, vias 1 -> 3
- net DIP2: track 12.6 -> 41.2 mm
- net PUSH: track 7.06 -> 19.5 mm
- net PWM-MOTOR-LEFT: track 70.2 -> 74.0 mm
- net DIP3: track 12.1 -> 14.9 mm
- net A15: track 20.8 -> 21.7 mm
- net A14: track 17.2 -> 18.1 mm

Commit message: Ruote Finish
Parts:
- moved FAN_AUX 9.68 mm to (98.4, 22.5)
- moved SW_FAN_AUX 5.43 mm to (92.7, 16.5), turned to 90 degrees
- moved SW_FAN1 4.60 mm to (92.7, 22.5), turned to 270 degrees
- moved Q2 2.92 mm to (94.4, 36.3)
- moved FAN1 2.54 mm to (98.4, 16.5), turned to 90 degrees
- moved LINE-SENSOR 2.08 mm to (87.0, 20.7)
- moved RLED-3 1.48 mm to (90.0, 67.8)
- moved RLED-4 1.48 mm to (93.2, 67.8)
- moved RLED-1 1.48 mm to (83.7, 67.8)
- moved RLED-2 1.48 mm to (86.9, 67.8)
- moved LED-PWR 1.27 mm to (83.3, 78.5)
- moved RPUSH-2 1.15 mm to (83.3, 75.7)
- moved RLED-PWR 1.14 mm to (83.4, 72.6)
- moved LED_1W 0.40 mm to (96.3, 29.1), turned to 270 degrees
Connections:
- net DIP3: now also ARDUINO-MEGA.26; no longer ARDUINO-MEGA.24
- net DIP4: now also ARDUINO-MEGA.24; no longer ARDUINO-MEGA.26
Routing:
- net GND: track 479.0 -> 523.5 mm
- net VCC: track 404.1 -> 422.9 mm
- net PUSH: track 19.5 -> 34.8 mm
- net 3V3: track 77.4 -> 90.9 mm, vias 3 -> 4
- net DIP3: track 14.9 -> 22.2 mm
- net N$15: track 4.34 -> 9.97 mm
- net N$128: track 18.7 -> 14.6 mm
- net N$1: track 6.13 -> 9.42 mm
- net N$2: track 4.84 -> 7.71 mm
- net IN1-MOTOR-LEFT: track 65.8 -> 62.9 mm
- net PWM-MOTOR-LEFT: track 74.0 -> 72.2 mm
- net OUT1-MOTOR-RIGHT: track 73.7 -> 75.4 mm
- net N$25: track 10.4 -> 11.7 mm
- net RX0: track 27.0 -> 28.2 mm
- net SCL: track 28.3 -> 27.1 mm
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
Commit message: Ruteo Ajustes
Parts:
- moved LED4 1.53 mm to (84.6, 53.7)
- moved R_BUZZ 1.14 mm to (84.5, 50.9)
- moved LED3 0.76 mm to (84.5, 56.4)
- moved DS1 0.52 mm to (84.3, 47.8)
- moved LED1 0.51 mm to (84.5, 61.5)
- moved DS4 0.36 mm to (84.2, 38.4)
- moved LED2 0.25 mm to (84.5, 58.8)
- moved DS3 0.18 mm to (84.3, 41.4)
- moved DS2 0.13 mm to (84.3, 44.5)
Connections:
- net VCC: now also DRIVER-LEFT.STBY, DRIVER-RIGHT.STBY
Routing:
- net VCC: track 422.9 -> 447.2 mm, vias 1 -> 2
- net PUSH: track 34.8 -> 21.1 mm
- net N$134: track 7.67 -> 17.6 mm, vias 0 -> 1
- net GND: track 523.5 -> 529.3 mm, vias 3 -> 4
- net ENC2-RIGHT: track 29.7 -> 28.4 mm
- net LED4: track 6.67 -> 5.59 mm
- net BUZZER: track 6.62 -> 5.56 mm
- net LED3: track 6.35 -> 5.44 mm
- net DIP4: track 19.7 -> 18.8 mm
- net LED2: track 6.16 -> 5.31 mm
- net N$6: track 14.6 -> 15.4 mm
- net DIP1: track 48.8 -> 49.5 mm
- net N$26: track 15.2 -> 15.8 mm
- added copper zone on layer 16, net GND2
- added copper zone on layer 1, net GND3
Other:
- board size 114.7 x 79.5 mm -> 114.7 x 79.4 mm

Commit message: Retoques
Parts:
- added U$1: LIPO7.4MOLEX, Baterias:KK-156-2
- moved BUZZER 9.70 mm to (103.1, 74.4), turned to 180 degrees
- moved ADXL335-ACELEROMETER 7.36 mm to (55.1, 76.1)
- moved PUSH-RST 7.07 mm to (54.4, 69.6)
- moved DIPSW 7.00 mm to (70.0, 72.9)
- moved DRIVER-LEFT 7.00 mm to (40.8, 49.4)
- moved DRIVER-RIGHT 7.00 mm to (40.8, 27.8)
- moved DS1 7.00 mm to (90.8, 45.1)
- moved DS2 7.00 mm to (90.8, 41.8)
- moved DS3 7.00 mm to (90.8, 38.7)
- moved DS4 7.00 mm to (90.7, 35.7)
- moved FAN1 7.00 mm to (104.9, 13.8)
- moved LED-PWR 7.00 mm to (89.8, 75.8)
- moved LED1 7.00 mm to (90.9, 58.8)
- moved LED2 7.00 mm to (90.9, 56.1)
- moved LED3 7.00 mm to (90.9, 53.7)
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Connections:
- removed net N$14: 5V-SOURCE.IN+, MOTORS-SOURCE.IN+, POWER-SW.P2
- net GND: now also U$1.GND
- net N$134: now also U$1.VCC
- net VIN: now also 5V-SOURCE.IN+, MOTORS-SOURCE.IN+, POWER-SW.P2
Routing:
- net VIN: track 0.00 -> 156.7 mm, vias 0 -> 1
- net N$14: track 76.5 -> 0.00 mm
- net GND: track 529.3 -> 553.1 mm
- net ENC2-LEFT: track 104.9 -> 99.8 mm
- net N$5: track 21.0 -> 16.1 mm
- net N$134: track 17.6 -> 22.3 mm
- net IN2-MOTOR-RIGHT: track 71.9 -> 67.8 mm
- net IN1-MOTOR-RIGHT: track 77.2 -> 74.5 mm
- net VCC: track 447.2 -> 449.9 mm
- net 6V-DC-3A: track 51.1 -> 53.7 mm
- net ENC1-LEFT: track 109.3 -> 107.3 mm
- net OUT2-MOTOR-RIGHT: track 70.8 -> 69.0 mm
- net PWM-MOTOR-RIGHT: track 67.3 -> 65.8 mm
- net 3V3: track 90.9 -> 91.8 mm
- net IN1-MOTOR-LEFT: track 62.9 -> 62.0 mm
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Other:
- board text added: "ProtecoHadware 2019"

Commit message: Shield Terminada
Parts:
- added C1: (no value), rcl:E5-10,5
- moved U$1 20.7 mm to (2.41, 73.3), turned to 90 degrees
- moved DRIVER-RIGHT 6.04 mm to (43.1, 22.2)
- moved SHARP-RIGHT 4.65 mm to (73.9, 3.68)
- moved SHARP-LEFT 4.51 mm to (52.7, 3.68)
- moved SHARP-MIDDLE 4.38 mm to (63.2, 3.68)
- moved POWER-SW 4.30 mm to (13.3, 73.0)
- moved PUSH-RST 4.19 mm to (56.8, 66.2)
- moved LED_1W 4.09 mm to (105.2, 23.1)
- moved LINE-SENSOR 4.09 mm to (95.9, 14.7)
- moved Q2 4.09 mm to (103.3, 30.4)
- moved R-DIP2 4.09 mm to (72.6, 53.2)
- moved RLED-3 4.09 mm to (98.9, 61.8)
- moved RLED-4 4.09 mm to (102.1, 61.8)
- moved U$9 4.09 mm to (74.5, 35.7)
- moved HC-05-PROG 4.09 mm to (34.9, 70.9)
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Connections:
- net GND: now also C1.-
- net VCC: now also C1.+
Routing:
- net GND: track 553.1 -> 584.7 mm
- net N$134: track 22.3 -> 42.6 mm, vias 1 -> 2
- net ENC1-LEFT: track 107.3 -> 100.8 mm
- net OUT2-MOTOR-RIGHT: track 69.0 -> 64.9 mm
- net IN2-MOTOR-LEFT: track 61.7 -> 58.3 mm
- net IN1-MOTOR-LEFT: track 62.0 -> 58.8 mm
- net OUT1-MOTOR-RIGHT: track 75.5 -> 72.5 mm
- net VCC: track 449.9 -> 452.9 mm
- net 3V3: track 91.8 -> 90.3 mm
- net OUT1-MOTOR-LEFT: track 84.1 -> 85.0 mm
- net IN1-MOTOR-RIGHT: track 74.5 -> 73.7 mm
- net INT: track 27.8 -> 28.5 mm
- net 6V-DC-3A: track 53.7 -> 54.3 mm
- net SHARP-RIGHT: track 16.4 -> 17.0 mm
- net RX2: track 20.8 -> 21.4 mm
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Other:
- board size 114.7 x 79.4 mm -> 114.9 x 81.3 mm
- board text added: "Acelerometer"
- board text added: "Bluetooth Programer"
- board text added: "Fan1"
- board text added: "Fan2"
- board text added: "Led1W"
- board text added: "Left"
- board text added: "M-Left"
- board text added: "Midd"
- board text added: "On ->"
- board text added: "PWR"
- board text added: "Proteco-Hadware"
- board text added: "Reset"
- board text added: "Right"
- board text added: "gnd"
- board text added: "vcc"
