File: Shield/Shield/Shield-Proteco.sch (EAGLE design)
At the start: 45 parts

Commit message: Programacion Inalambrica con BT
Parts:
- removed SW2: (no value), special:SW_DIP-1
- removed U$13: HC-05-PROG, hc-xx:HC-05-PROG
- added LED6: (no value), led:LEDCHIPLED_1206
- added R15: (no value), rcl:R-US_M1206
- added SHARP-LEFT, SHARP-MIDDLE: SHARP, Sensores:SHARP
- added U$18: SLIDE-3, Interruptores:SLIDE-3
- U$10: value SHARP -> SERVOMOTORES; device Sensores:SHARP -> Motores:SERVOMOTORES
- U$9: value SHARP -> SENSOR-MISCELANEOUS; device Sensores:SHARP -> Sensores:SENSOR-MISCELANEOUS
- renumbered SG1 to BUZZER, T1 to BC547, U$11 to SHARP-RIGHT
Connections:
- removed net N$16: SW2.1, U$13.RESET
- removed net RX0: U$13.RX
- removed net TX0: U$13.TX
- new net LED1: LED1.A
- new net LED2: LED2.A
- new net LED3: LED3.A
- new net LED4: LED4.A
- new net LED5: LED5.A
- new net N$100: U$3.AO2, U$3.BO2
- new net N$101: U$3.AO1, U$3.BO1
- new net N$102: U$7.OUTB
- new net N$103: U$7.OUTA
- new net N$104: U$7.M2
- new net N$105: U$7.M1
- new net N$106: U$8.OUTA
- new net N$107: U$8.OUTB
- new net N$108: U$8.M2
- new net N$109: U$8.M1
- new net N$110: U$9.3.3V
- new net N$111: ARDUINO-MEGA.12
- new net N$112: ARDUINO-MEGA.11
- new net N$113: ARDUINO-MEGA.10
- new net N$114: ARDUINO-MEGA.9
- new net N$115: ARDUINO-MEGA.8
- new net N$116: ARDUINO-MEGA.7
- new net N$117: ARDUINO-MEGA.6
- new net N$75: U$1.SIGNAL
- new net N$76: U$16.SIGNAL
- new net N$77: U$10.SIGNAL, U$17.SIGNAL
- new net N$78: ARDUINO-MEGA.SCL
- new net N$79: ARDUINO-MEGA.SDA
- new net N$80: ARDUINO-MEGA.AREF
- new net N$81: ARDUINO-MEGA.GND
- new net N$82: U$9.E2
- new net N$83: U$9.E3
- new net N$84: U$9.E4
- new net N$85: U$9.E5
- new net N$86: U$9.E6
- new net N$87: U$9.E7
- new net N$88: LED5.C, R14.2
- new net N$89: LED6.C, R15.2
- new net N$92: U$6.AIN1, U$6.BIN1
- new net N$93: U$6.AIN2, U$6.BIN2
- new net N$94: U$6.AO2, U$6.BO2
- new net N$95: U$6.AO1, U$6.BO1
- new net N$96: U$6.PWMA, U$6.PWMB
- new net N$97: U$3.AIN1, U$3.BIN1
- new net N$98: U$3.AIN2, U$3.BIN2
- new net N$99: U$3.PWMA, U$3.PWMB
- new net SD_SCK: ARDUINO-MEGA.13, U$14.SD_SCK
- net GND: now also R15.1, SHARP-LEFT.GND, SHARP-MIDDLE.GND; no longer U$13.GND
- net N$10: now also S2.P1
- net N$11: now also S1.P1
- net N$12: now also S3.P1
- net N$13: now also S4.P1
- net N$29: now also U$18.P2
- net N$69: now also U$9.E1; no longer U$14.SD_SCK
- net N$7: now also SHARP-LEFT.DISTANCE; no longer U$9.DISTANCE
- net N$8: now also SHARP-MIDDLE.DISTANCE; no longer U$10.DISTANCE
- net RESET: no longer SW2.2
- net VCC: now also LED6.A, SHARP-LEFT.VCC, SHARP-MIDDLE.VCC, U$18.COM; no longer U$13.VCC
Other:
- moved on the sheet: R1, R2, R3, R4

Commit message: Más avance
Parts:
- added D1, D2, D3, D4: (no value), diode:DIODE-DO-214AC
- added Q1: FDD4141TO252, transistor-fet:FDD4141TO252
- added U$11: ACELEROMETER-JST-5, Sensores:ACELEROMETER-JST-5
- added U$13: HC-05-PROGRAMER, hc-xx:HC-05-PROGRAMER
- added U$19: SW-HEAD, Interruptores:SW-HEAD
- added U$20, U$21: FAN-MOLEX, Ventilador:FAN-MOLEX
- added U$22: LED-1W-3V3, LedPower:LED-1W-3V3
- added U$23: ZIIPY-7.4V, Baterias:ZIIPY-7.4V
- U$12: value CNY70-ARRAY -> CNY70-ARRAY-HEADER; device Sensores:CNY70-ARRAY -> Sensores:CNY70-ARRAY-HEADER
- U$15: value ACELEROMETER-MPU6050-JST -> SLIDE-3; device Sensores:ACELEROMETER-MPU6050-JST -> Interruptores:SLIDE-3
- U$18: value SLIDE-3 -> SW-HEAD; device Interruptores:SLIDE-3 -> Interruptores:SW-HEAD
Connections:
- new net DRAIN: Q1.D
- new net GATE: Q1.G
- new net N$118: ARDUINO-MEGA.0-RX0
- new net N$119: ARDUINO-MEGA.14-TX3
- new net N$120: ARDUINO-MEGA.15-RX3
- new net N$121: ARDUINO-MEGA.16-TX2
- new net N$122: ARDUINO-MEGA.17-RX2
- new net N$123: ARDUINO-MEGA.18-TX1
- new net N$124: ARDUINO-MEGA.19-RX1
- new net N$125: ARDUINO-MEGA.20-SDA
- new net N$126: ARDUINO-MEGA.21-SCL
- new net N$127: D1.A, U$1.SIGNAL
- new net N$128: U$18.2, U$20.VCC
- new net N$129: U$9.E9
- new net N$130: U$9.E10
- new net N$131: U$9.E11
- new net N$132: U$9.E12
- new net N$133: U$9.E13
- new net N$134: U$2.1, U$23.7.4V
- new net N$16: ARDUINO-MEGA.5
- new net N$90: ARDUINO-MEGA.1-TX0
- new net N$91: U$13.RX
- new net RX0: U$13.TX
- new net SERVO1: D1.C
- new net SERVO2: D2.C
- new net SERVO3: D3.C
- new net SERVO4: D4.C
- new net SOURCE: Q1.S
- net GND: now also U$11.GND, U$13.GND, U$20.GND, U$21.GND, U$23.GND; no longer U$15.GND
- net N$14: now also U$2.2; no longer U$2.P2
- net N$15: now also U$19.2, U$21.VCC; no longer U$2.COM
- net N$17: now also U$11.SCL; no longer U$15.SCL
- net N$18: now also U$11.SDA; no longer U$15.SDA
- net N$19: now also ARDUINO-MEGA.4; no longer U$15.XDA
- net N$20: now also ARDUINO-MEGA.3; no longer U$15.XCL
- net N$21: now also ARDUINO-MEGA.2; no longer U$15.ADO
- net N$22: now also U$11.INT; no longer U$15.INT
- net N$29: now also U$15.2; no longer U$18.P2
- net N$75: now also D4.A, U$10.SIGNAL; no longer U$1.SIGNAL
- net N$76: now also D3.A, U$17.SIGNAL; no longer U$16.SIGNAL
- net N$77: now also D2.A, U$16.SIGNAL; no longer U$10.SIGNAL, U$17.SIGNAL
- net RESET: now also U$13.RESET
- net VCC: now also U$11.VCC, U$13.VCC, U$15.COM, U$18.1, U$19.1; no longer U$15.VCC, U$18.COM
Other:
- moved on the sheet: ARDUINO-MEGA, BC547, BUZZER, R1, R2, R3, R4, R5, SHARP-LEFT, SHARP-MIDDLE, SHARP-RIGHT, SW1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

Commit message: Name
Connections:
- net N$39 renamed 3V3
- removed net N$41: ARDUINO-MEGA.GND_2
- net GND: now also ARDUINO-MEGA.GND_2
Changed lines of the file:
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@@
 <setting verticaltext="up"/>
 </settings>
-<grid distance="0.05" unitdist="inch" unit="inch" style="lines" multiple="1" display="yes" altdistance="0.01" altunitdist="inch" altunit="inch"/>
+<grid distance="0.1" unitdist="inch" unit="inch" style="lines" multiple="1" display="no" altdistance="0.01" altunitdist="inch" altunit="inch"/>
 <layers>
 <layer number="1" name="Top" color="4" fill="1" visible="no" active="no"/>
@@
 <wire x1="-316.23" y1="180.34" x2="-316.23" y2="175.26" width="0.1524" layer="91"/>
 </segment>
+<segment>
+<pinref part="ARDUINO-MEGA" gate="G$1" pin="GND_2"/>
+<wire x1="46.99" y1="-15.24" x2="29.21" y2="-15.24" width="0.1524" layer="91"/>
+<label x="29.21" y="-15.24" size="1.778" layer="95" rot="R180" xref="yes"/>
+</segment>
 </net>
 <net name="N$5" class="0">
@@
 </segment>
 </net>
-<net name="N$39" class="0">
+<net name="3V3" class="0">
 <segment>
 <pinref part="ARDUINO-MEGA" gate="G$1" pin="3V3"/>
@@
 </segment>
 </net>
-<net name="N$41" class="0">
-<segment>
-<pinref part="ARDUINO-MEGA" gate="G$1" pin="GND_2"/>
-<wire x1="46.99" y1="-15.24" x2="29.21" y2="-15.24" width="0.1524" layer="91"/>
-<label x="29.21" y="-15.24" size="1.778" layer="95" rot="R180" xref="yes"/>
-</segment>
-</net>

Commit message: Conexiones
Parts:
- removed R6, R7, R8, R9: (no value), rcl:R-US_M1206
- removed S1, S2, S3, S4: (no value), switch-omron:10-XX
- added PUSH-RST, PUSH2, PUSH3, PUSH4: (no value), switch-omron:10-XX
- added R-PUSH3, RPUSH-2, RPUSH-4: (no value), rcl:R-US_M1206
- renumbered D1 to DS1, D2 to DS2, D3 to DS3, D4 to DS4, LED6 to LED-PWR, R1 to R-DIP1, R10 to RLED-1, R11 to RLED-2, R12 to RLED-3, R13 to RLED-4, R14 to RLED-5, R15 to RLED-PWR, R2 to R-DIP2, R3 to R-DIP3, R4 to R-DIP4, R5 to R_BUZZ, SW1 to DIPSW, U$1 to SERVO_1, U$10 to SERVO_4, U$11 to ADXL335-ACELEROMETER, U$12 to LINE-SENSOR, U$13 to HC-05-PROG, U$15 to TFT-SW, U$16 to SERVO_2, U$17 to SERVO_3, U$18 to SW_FAN1, U$19 to SW_FAN_AUX, U$2 to POWER-SW, U$20 to FAN1, U$21 to FAN_AUX, U$22 to LED_1W, U$3 to DRIVER-RIGHT, U$4 to 5V-SOURCE, U$5 to MOTORS-SOURCE, U$6 to DRIVER-LEFT, U$7 to MOTOR_LEFT, U$8 to MOTOR_RIGHT
Connections:
- net N$1 renamed DIP1
- net N$2 renamed DIP2
- net N$22 renamed INT
- net N$3 renamed DIP3
- net N$32 renamed VIN
- net N$4 renamed DIP4
- net N$7 renamed SHARP-LEFT
- net N$70 renamed SD_DO
- net N$71 renamed SD_DI
- net N$72 renamed SD_SS
- net N$73 renamed LCD_D1
- net N$74 renamed LCD_D0
- net N$8 renamed SHARP-MIDDLE
- net N$9 renamed SHARP-RIGHT
- net N$92 renamed IN1-MOTOR-LEFT
- net N$93 renamed IN2-MOTOR-LEFT
- net N$96 renamed PWM-MOTOR-LEFT
- net N$97 renamed IN2-MOTOR-RIGHT
- net N$98 renamed IN1-MOTOR-RIGHT
- net N$99 renamed PWM-MOTOR-RIGHT
- removed net N$10: R7.2, S2.P, S2.P1
- removed net N$100: DRIVER-RIGHT.AO2, DRIVER-RIGHT.BO2
- removed net N$101: DRIVER-RIGHT.AO1, DRIVER-RIGHT.BO1
- removed net N$102: MOTOR_LEFT.OUTB
- removed net N$103: MOTOR_LEFT.OUTA
- removed net N$106: MOTOR_RIGHT.OUTA
- removed net N$107: MOTOR_RIGHT.OUTB
- removed net N$11: R6.2, S1.P, S1.P1
- removed net N$110: U$9.3.3V
- removed net N$116: ARDUINO-MEGA.7
- removed net N$117: ARDUINO-MEGA.6
- removed net N$118: ARDUINO-MEGA.0-RX0
- removed net N$12: R8.2, S3.P, S3.P1
- removed net N$13: R9.2, S4.P, S4.P1
- removed net N$16: ARDUINO-MEGA.5
- removed net N$17: ADXL335-ACELEROMETER.SCL
- removed net N$18: ADXL335-ACELEROMETER.SDA
- removed net N$19: ARDUINO-MEGA.4
- removed net N$20: ARDUINO-MEGA.3
- removed net N$21: ARDUINO-MEGA.2
- removed net N$27: U$14.NC_5
- removed net N$28: U$14.3V3
- removed net N$33: U$14.LCD_RD
- removed net N$34: U$14.LCD_WR
- removed net N$35: U$14.LCD_RS
- removed net N$36: U$14.LCD_CS
- removed net N$37: U$14.LCD_RST
- removed net N$44: ARDUINO-MEGA.A0
- removed net N$45: ARDUINO-MEGA.A1
- removed net N$46: ARDUINO-MEGA.A2
- removed net N$47: ARDUINO-MEGA.A3
- removed net N$48: ARDUINO-MEGA.A4
- removed net N$60: U$14.NC_6
- removed net N$61: U$14.LCD_D2
- removed net N$62: U$14.LCD_D3
- removed net N$63: U$14.LCD_D4
- removed net N$64: U$14.LCD_D5
- removed net N$65: U$14.LCD_D6
- removed net N$66: U$14.LCD_D7
- removed net N$68: U$14.NC_7
- removed net N$78: ARDUINO-MEGA.SCL
- removed net N$79: ARDUINO-MEGA.SDA
- removed net N$81: ARDUINO-MEGA.GND
- removed net N$90: ARDUINO-MEGA.1-TX0
- removed net N$91: HC-05-PROG.RX
- removed net N$94: DRIVER-LEFT.AO2, DRIVER-LEFT.BO2
- removed net N$95: DRIVER-LEFT.AO1, DRIVER-LEFT.BO1
- new net LCD_CS: ARDUINO-MEGA.A3, U$14.LCD_CS
- new net LCD_D2: ARDUINO-MEGA.2, U$14.LCD_D2
- new net LCD_D3: ARDUINO-MEGA.3, U$14.LCD_D3
- new net LCD_D4: ARDUINO-MEGA.4, U$14.LCD_D4
- new net LCD_D5: ARDUINO-MEGA.5, U$14.LCD_D5
- new net LCD_D6: ARDUINO-MEGA.6, U$14.LCD_D6
- new net LCD_D7: ARDUINO-MEGA.7, U$14.LCD_D7
- new net LCD_RD: ARDUINO-MEGA.A0, U$14.LCD_RD
- new net LCD_RS: ARDUINO-MEGA.A2, U$14.LCD_RS
- new net LCD_RST: ARDUINO-MEGA.A4, U$14.LCD_RST
- new net LCD_WR: ARDUINO-MEGA.A1, U$14.LCD_WR
- new net OUT1-MOTOR-LEFT: DRIVER-LEFT.AO1, DRIVER-LEFT.BO1, MOTOR_LEFT.OUTB
- new net OUT1-MOTOR-RIGHT: DRIVER-RIGHT.AO1, DRIVER-RIGHT.BO1, MOTOR_RIGHT.OUTB
- new net OUT2-MOTOR-LEFT: DRIVER-LEFT.AO2, DRIVER-LEFT.BO2, MOTOR_LEFT.OUTA
- new net OUT2-MOTOR-RIGHT: DRIVER-RIGHT.AO2, DRIVER-RIGHT.BO2, MOTOR_RIGHT.OUTA
- new net PUSH2: PUSH2.P, PUSH2.P1, RPUSH-2.2
- new net PUSH3: PUSH3.P, PUSH3.P1, R-PUSH3.2
- new net PUSH4: PUSH4.P, PUSH4.P1, RPUSH-4.2
- new net SCL: ADXL335-ACELEROMETER.SCL, ARDUINO-MEGA.SCL
- new net SDA: ADXL335-ACELEROMETER.SDA, ARDUINO-MEGA.SDA
- new net TX0: ARDUINO-MEGA.1-TX0, HC-05-PROG.RX, U$14.NC_6
- net 3V3: now also U$14.3V3, U$9.3.3V
- net GND: now also ARDUINO-MEGA.GND, R-PUSH3.1, RPUSH-2.1, RPUSH-4.1, U$14.NC_7; no longer R6.1, R7.1, R8.1, R9.1
- net RESET: now also PUSH-RST.P, PUSH-RST.P1
- net RX0: now also ARDUINO-MEGA.0-RX0, U$14.NC_5
- net VCC: now also PUSH-RST.S, PUSH2.S, PUSH3.S, PUSH4.S; no longer S1.S, S2.S, S3.S, S4.S

Commit message: Conexiones+
Parts:
- removed TFT-SW: SLIDE-3, Interruptores:SLIDE-3
Connections:
- removed net N$111: ARDUINO-MEGA.12
- removed net N$112: ARDUINO-MEGA.11
- removed net N$113: ARDUINO-MEGA.10
- removed net N$114: ARDUINO-MEGA.9
- removed net N$115: ARDUINO-MEGA.8
- removed net N$29: TFT-SW.2, U$14.5V
- removed net N$30: U$14.NC_3
- removed net N$31: U$14.GND
- removed net N$40: ARDUINO-MEGA.5V_1
- removed net N$42: ARDUINO-MEGA.GND_1
- removed net N$43: ARDUINO-MEGA.VIN
- removed net N$67: U$14.NC_8
- removed net N$80: ARDUINO-MEGA.AREF
- new net AREF: ARDUINO-MEGA.AREF, U$14.NC_8
- net GND: now also ARDUINO-MEGA.GND_1, U$14.GND, U$14.NC_3
- net LCD_D0: now also ARDUINO-MEGA.8
- net LCD_D1: now also ARDUINO-MEGA.9
- net N$134: now also POWER-SW.COM; no longer POWER-SW.1
- net SD_DI: now also ARDUINO-MEGA.11
- net SD_DO: now also ARDUINO-MEGA.12
- net SD_SS: now also ARDUINO-MEGA.10
- net VCC: now also ARDUINO-MEGA.5V_1, U$14.5V; no longer TFT-SW.COM
- net VIN: now also ARDUINO-MEGA.VIN

Commit message: Disposicion de pines
Parts:
- removed LED5: (no value), led:LEDCHIPLED_1206
- removed PUSH3, PUSH4: (no value), switch-omron:10-XX
- removed R-PUSH3, RLED-5, RPUSH-4: (no value), rcl:R-US_M1206
Connections:
- removed net LED5: LED5.A
- removed net N$88: LED5.C, RLED-5.2
- removed net PUSH3: PUSH3.P, PUSH3.P1, R-PUSH3.2
- removed net PUSH4: PUSH4.P, PUSH4.P1, RPUSH-4.2
- new net N$1: U$9.E8
- net GND: no longer R-PUSH3.1, RLED-5.1, RPUSH-4.1
- net VCC: no longer PUSH3.S, PUSH4.S
Changed lines of the file:
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@@
 <part name="PUSH-RST" library="switch-omron" library_urn="urn:adsk.eagle:library:377" deviceset="10-XX" device="" package3d_urn="urn:adsk.eagle:package:27496/1"/>
 <part name="PUSH2" library="switch-omron" library_urn="urn:adsk.eagle:library:377" deviceset="10-XX" device="" package3d_urn="urn:adsk.eagle:package:27496/1"/>
-<part name="PUSH3" library="switch-omron" library_urn="urn:adsk.eagle:library:377" deviceset="10-XX" device="" package3d_urn="urn:adsk.eagle:package:27496/1"/>
-<part name="PUSH4" library="switch-omron" library_urn="urn:adsk.eagle:library:377" deviceset="10-XX" device="" package3d_urn="urn:adsk.eagle:package:27496/1"/>
 <part name="RPUSH-2" library="rcl" library_urn="urn:adsk.eagle:library:334" deviceset="R-US_" device="M1206" package3d_urn="urn:adsk.eagle:package:23566/1"/>
-<part name="R-PUSH3" library="rcl" library_urn="urn:adsk.eagle:library:334" deviceset="R-US_" device="M1206" package3d_urn="urn:adsk.eagle:package:23566/1"/>
-<part name="RPUSH-4" library="rcl" library_urn="urn:adsk.eagle:library:334" deviceset="R-US_" device="M1206" package3d_urn="urn:adsk.eagle:package:23566/1"/>
 <part name="GND9" library="supply1" library_urn="urn:adsk.eagle:library:371" deviceset="GND" device=""/>
-<part name="GND10" library="supply1" library_urn="urn:adsk.eagle:library:371" deviceset="GND" device=""/>
-<part name="GND11" library="supply1" library_urn="urn:adsk.eagle:library:371" deviceset="GND" device=""/>
 <part name="P+8" library="supply1" library_urn="urn:adsk.eagle:library:371" deviceset="VCC" device=""/>
 <part name="P+9" library="supply1" library_urn="urn:adsk.eagle:library:371" deviceset="VCC" device=""/>
-<part name="P+10" library="supply1" library_urn="urn:adsk.eagle:library:371" deviceset="VCC" device=""/>
-<part name="P+11" library="supply1" library_urn="urn:adsk.eagle:library:371" deviceset="VCC" device=""/>
 <part name="GND12" library="supply1" library_urn="urn:adsk.eagle:library:371" deviceset="GND" device=""/>
 <part name="GND13" library="supply1" library_urn="urn:adsk.eagle:library:371" deviceset="GND" device=""/>
@@
 <part name="LED3" library="led" library_urn="urn:adsk.eagle:library:259" deviceset="LED" device="CHIPLED_1206" package3d_urn="urn:adsk.eagle:package:15823/2"/>
 <part name="LED4" library="led" library_urn="urn:adsk.eagle:library:259" deviceset="LED" device="CHIPLED_1206" package3d_urn="urn:adsk.eagle:package:15823/2"/>
-<part name="LED5" library="led" library_urn="urn:adsk.eagle:library:259" deviceset="LED" device="CHIPLED_1206" package3d_urn="urn:adsk.eagle:package:15823/2"/>
 <part name="RLED-1" library="rcl" library_urn="urn:adsk.eagle:library:334" deviceset="R-US_" device="M1206" package3d_urn="urn:adsk.eagle:package:23566/1"/>
 <part name="RLED-2" library="rcl" library_urn="urn:adsk.eagle:library:334" deviceset="R-US_" device="M1206" package3d_urn="urn:adsk.eagle:package:23566/1"/>
 <part name="RLED-3" library="rcl" library_urn="urn:adsk.eagle:library:334" deviceset="R-US_" device="M1206" package3d_urn="urn:adsk.eagle:package:23566/1"/>
 <part name="RLED-4" library="rcl" library_urn="urn:adsk.eagle:library:334" deviceset="R-US_" device="M1206" package3d_urn="urn:adsk.eagle:package:23566/1"/>
-<part name="RLED-5" library="rcl" library_urn="urn:adsk.eagle:library:334" deviceset="R-US_" device="M1206" package3d_urn="urn:adsk.eagle:package:23566/1"/>
 <part name="GND23" library="supply1" library_urn="urn:adsk.eagle:library:371" deviceset="GND" device=""/>
 <part name="GND24" library="supply1" library_urn="urn:adsk.eagle:library:371" deviceset="GND" device=""/>
 <part name="GND25" library="supply1" library_urn="urn:adsk.eagle:library:371" deviceset="GND" device=""/>
 <part name="GND26" library="supply1" library_urn="urn:adsk.eagle:library:371" deviceset="GND" device=""/>
-<part name="GND27" library="supply1" library_urn="urn:adsk.eagle:library:371" deviceset="GND" device=""/>
 <part name="SERVO_1" library="Motores" deviceset="SERVOMOTORES" device=""/>
 <part name="SERVO_2" library="Motores" deviceset="SERVOMOTORES" device=""/>
@@
 <instance part="PUSH-RST" gate="1" x="-165.1" y="133.35"/>
 <instance part="PUSH2" gate="1" x="-138.43" y="133.35"/>
-<instance part="PUSH3" gate="1" x="-111.76" y="133.35"/>
-<instance part="PUSH4" gate="1" x="-83.82" y="133.35"/>
 <instance part="RPUSH-2" gate="G$1" x="-138.43" y="121.92" rot="R90"/>
-<instance part="R-PUSH3" gate="G$1" x="-111.76" y="121.92" rot="R90"/>
-<instance part="RPUSH-4" gate="G$1" x="-83.82" y="121.92" rot="R90"/>
 <instance part="GND9" gate="1" x="-138.43" y="114.3"/>
-<instance part="GND10" gate="1" x="-111.76" y="114.3"/>
-<instance part="GND11" gate="1" x="-83.82" y="114.3"/>
 <instance part="P+8" gate="VCC" x="-165.1" y="143.51"/>
 <instance part="P+9" gate="VCC" x="-138.43" y="143.51"/>
-<instance part="P+10" gate="VCC" x="-111.76" y="143.51"/>
-<instance part="P+11" gate="VCC" x="-83.82" y="143.51"/>
 <instance part="GND12" gate="1" x="-238.76" y="129.54"/>
 <instance part="GND13" gate="1" x="-105.41" y="-1.27"/>
@@
 <instance part="LED3" gate="G$1" x="-120.65" y="185.42"/>
 <instance part="LED4" gate="G$1" x="-109.22" y="185.42"/>
-<instance part="LED5" gate="G$1" x="-97.79" y="185.42"/>
 <instance part="RLED-1" gate="G$1" x="-148.59" y="172.72" rot="R90"/>
 <instance part="RLED-2" gate="G$1" x="-134.62" y="172.72" rot="R90"/>
 <instance part="RLED-3" gate="G$1" x="-120.65" y="172.72" rot="R90"/>
 <instance part="RLED-4" gate="G$1" x="-109.22" y="172.72" rot="R90"/>
-<instance part="RLED-5" gate="G$1" x="-97.79" y="172.72" rot="R90"/>
 <instance part="GND23" gate="1" x="-148.59" y="165.1"/>
 <instance part="GND24" gate="1" x="-134.62" y="165.1"/>
 <instance part="GND25" gate="1" x="-120.65" y="165.1"/>
 <instance part="GND26" gate="1" x="-109.22" y="165.1"/>
-<instance part="GND27" gate="1" x="-97.79" y="165.1"/>
 <instance part="SERVO_1" gate="G$1" x="-119.38" y="-142.24"/>
 <instance part="SERVO_2" gate="G$1" x="-119.38" y="-172.72"/>
@@
 <instance part="P+24" gate="VCC" x="-97.79" y="-223.52"/>
 <instance part="GND33" gate="1" x="-99.06" y="-238.76"/>
-<instance part="LOGO1" gate="G$1" x="262.89" y="173.99"/>
+<instance part="LOGO1" gate="G$1" x="224.79" y="-284.48"/>
 <instance part="ADXL335-ACELEROMETER" gate="G$1" x="80.01" y="156.21"/>
 <instance part="HC-05-PROG" gate="G$1" x="-35.56" y="154.94"/>
@@
 </segment>
 <segment>
-<pinref part="PUSH3" gate="1" pin="S"/>
-<pinref part="P+10" gate="VCC" pin="VCC"/>
-<wire x1="-111.76" y1="138.43" x2="-111.76" y2="140.97" width="0.1524" layer="91"/>
-</segment>
-<segment>
-<pinref part="PUSH4" gate="1" pin="S"/>
-<pinref part="P+11" gate="VCC" pin="VCC"/>
-<wire x1="-83.82" y1="138.43" x2="-83.82" y2="140.97" width="0.1524" layer="91"/>
-</segment>
-<segment>
 <pinref part="P+12" gate="VCC" pin="VCC"/>
 <wire x1="-33.02" y1="125.73" x2="-21.59" y2="125.73" width="0.1524" layer="91"/>
@@
 </segment>
 <segment>
-<pinref part="R-PUSH3" gate="G$1" pin="1"/>
-<pinref part="GND10" gate="1" pin="GND"/>
-</segment>
-<segment>
-<pinref part="RPUSH-4" gate="G$1" pin="1"/>
-<pinref part="GND11" gate="1" pin="GND"/>
-</segment>
-<segment>
 <pinref part="GND12" gate="1" pin="GND"/>
 <wire x1="-242.57" y1="137.16" x2="-242.57" y2="132.08" width="0.1524" layer="91"/>
@@
 <pinref part="RLED-4" gate="G$1" pin="1"/>
 <pinref part="GND26" gate="1" pin="GND"/>
-</segment>
-<segment>
-<pinref part="RLED-5" gate="G$1" pin="1"/>
-<pinref part="GND27" gate="1" pin="GND"/>
 </segment>
 <segment>
@@
 </segment>
 </net>
-<net name="PUSH3" class="0">
-<segment>
-<pinref part="PUSH3" gate="1" pin="P"/>
-<pinref part="R-PUSH3" gate="G$1" pin="2"/>
-<wire x1="-111.76" y1="127" x2="-109.22" y2="128.27" width="0.1524" layer="91"/>
-<junction x="-111.76" y="127"/>
-<label x="-105.41" y="128.27" size="1.778" layer="95" xref="yes"/>
-<pinref part="PUSH3" gate="1" pin="P1"/>
-<wire x1="-109.22" y1="128.27" x2="-105.41" y2="128.27" width="0.1524" layer="91"/>
-<junction x="-109.22" y="128.27"/>
-<wire x1="-111.76" y1="127" x2="-111.76" y2="128.27" width="0.1524" layer="91"/>
-</segment>
-</net>
-<net name="PUSH4" class="0">
-<segment>
-<pinref part="PUSH4" gate="1" pin="P"/>
-<pinref part="RPUSH-4" gate="G$1" pin="2"/>
-<wire x1="-83.82" y1="127" x2="-81.28" y2="128.27" width="0.1524" layer="91"/>
-<junction x="-83.82" y="127"/>
-<label x="-77.47" y="128.27" size="1.778" layer="95" xref="yes"/>
-<pinref part="PUSH4" gate="1" pin="P1"/>
-<wire x1="-81.28" y1="128.27" x2="-77.47" y2="128.27" width="0.1524" layer="91"/>
-<junction x="-81.28" y="128.27"/>
-<wire x1="-83.82" y1="127" x2="-83.82" y2="128.27" width="0.1524" layer="91"/>
-</segment>
-</net>
 <net name="N$14" class="0">
 <segment>
@@
 <wire x1="-114.3" y1="187.96" x2="-114.3" y2="193.04" width="0.1524" layer="91"/>
 <label x="-114.3" y="193.04" size="1.778" layer="95" rot="R90" xref="yes"/>
-</segment>
-</net>
-<net name="LED5" class="0">
-<segment>
-<pinref part="LED5" gate="G$1" pin="A"/>
-<wire x1="-97.79" y1="187.96" x2="-101.6" y2="187.96" width="0.1524" layer="91"/>
-<wire x1="-101.6" y1="187.96" x2="-101.6" y2="193.04" width="0.1524" layer="91"/>
-<label x="-101.6" y="193.04" size="1.778" layer="95" rot="R90" xref="yes"/>
-</segment>
-</net>
-<net name="N$88" class="0">
-<segment>
-<pinref part="RLED-5" gate="G$1" pin="2"/>
-<pinref part="LED5" gate="G$1" pin="C"/>
-<wire x1="-97.79" y1="177.8" x2="-97.79" y2="180.34" width="0.1524" layer="91"/>
 </segment>
 </net>
@@
 </segment>
 </net>
+<net name="N$1" class="0">
+<segment>
+<pinref part="U$9" gate="G$1" pin="E8"/>
+<wire x1="284.48" y1="-102.87" x2="267.97" y2="-102.87" width="0.1524" layer="91"/>
+<label x="267.97" y="-102.87" size="1.778" layer="95" rot="R180" xref="yes"/>
+</segment>
+</net>
