File: Shield/Shield/Shield-Proteco.sch (EAGLE design)
At the start: 52 parts, among them Q1 FDD4141TO252

Commit message: Conexiones
Parts:
- renumbered PUSH2 to PUSH
Connections:
- removed net N$1: U$9.E8
- removed net N$104: MOTOR_LEFT.M2
- removed net N$105: MOTOR_LEFT.M1
- removed net N$108: MOTOR_RIGHT.M2
- removed net N$109: MOTOR_RIGHT.M1
- removed net N$119: ARDUINO-MEGA.14-TX3
- removed net N$120: ARDUINO-MEGA.15-RX3
- removed net N$121: ARDUINO-MEGA.16-TX2
- removed net N$122: ARDUINO-MEGA.17-RX2
- removed net N$123: ARDUINO-MEGA.18-TX1
- removed net N$124: ARDUINO-MEGA.19-RX1
- removed net N$125: ARDUINO-MEGA.20-SDA
- removed net N$126: ARDUINO-MEGA.21-SCL
- removed net N$129: U$9.E9
- removed net N$130: U$9.E10
- removed net N$131: U$9.E11
- removed net N$132: U$9.E12
- removed net N$133: U$9.E13
- removed net N$49: ARDUINO-MEGA.A5
- removed net N$50: ARDUINO-MEGA.A6
- removed net N$51: ARDUINO-MEGA.A7
- removed net N$52: ARDUINO-MEGA.A8
- removed net N$53: ARDUINO-MEGA.A9
- removed net N$54: ARDUINO-MEGA.A10
- removed net N$55: ARDUINO-MEGA.A11
- removed net N$56: ARDUINO-MEGA.A12
- removed net N$57: ARDUINO-MEGA.A13
- removed net N$58: ARDUINO-MEGA.A14
- removed net N$59: ARDUINO-MEGA.A15
- removed net N$69: U$9.E1
- removed net N$82: U$9.E2
- removed net N$83: U$9.E3
- removed net N$84: U$9.E4
- removed net N$85: U$9.E5
- removed net N$86: U$9.E6
- removed net N$87: U$9.E7
- removed net PUSH2: PUSH.P, PUSH.P1, RPUSH-2.2
- new net A10: ARDUINO-MEGA.A10, U$9.E4
- new net A11: ARDUINO-MEGA.A11, U$9.E5
- new net A12: ARDUINO-MEGA.A12, U$9.E6
- new net A13: ARDUINO-MEGA.A13, U$9.E7
- new net A14: ARDUINO-MEGA.A14, U$9.E8
- new net A15: ARDUINO-MEGA.A15, U$9.E9
- new net A9: ARDUINO-MEGA.A9, U$9.E3
- new net D36: ARDUINO-MEGA.36, U$9.E10
- new net D38: ARDUINO-MEGA.38, U$9.E11
- new net D40: ARDUINO-MEGA.40, U$9.E12
- new net D42: ARDUINO-MEGA.42, U$9.E13
- new net ENC1-LEFT: ARDUINO-MEGA.14-TX3, MOTOR_LEFT.M1
- new net ENC1-RIGHT: ARDUINO-MEGA.18-TX1, MOTOR_RIGHT.M1
- new net ENC2-LEFT: ARDUINO-MEGA.15-RX3, MOTOR_LEFT.M2
- new net ENC2-RIGHT: ARDUINO-MEGA.A8, MOTOR_RIGHT.M2
- new net LED1W: ARDUINO-MEGA.45
- new net N$10: ARDUINO-MEGA.49
- new net N$11: ARDUINO-MEGA.51
- new net N$12: ARDUINO-MEGA.53
- new net N$33: ARDUINO-MEGA.50
- new net N$42: ARDUINO-MEGA.48
- new net N$43: ARDUINO-MEGA.52
- new net PUSH: ARDUINO-MEGA.25, PUSH.P, PUSH.P1, RPUSH-2.2
- new net RX2: ARDUINO-MEGA.17-RX2, U$9.E1
- new net TX2: ARDUINO-MEGA.16-TX2, U$9.E2
- net BUZZER: now also ARDUINO-MEGA.35
- net DIP1: now also ARDUINO-MEGA.23
- net DIP2: now also ARDUINO-MEGA.22, ARDUINO-MEGA.5V_3
- net DIP3: now also ARDUINO-MEGA.24
- net DIP4: now also ARDUINO-MEGA.26
- net INT: now also ARDUINO-MEGA.19-RX1
- net LED1: now also ARDUINO-MEGA.27
- net LED2: now also ARDUINO-MEGA.29
- net LED3: now also ARDUINO-MEGA.31
- net LED4: now also ARDUINO-MEGA.33
- net OUT1-MOTOR-LEFT: now also ARDUINO-MEGA.28
- net OUT1-MOTOR-RIGHT: now also ARDUINO-MEGA.32
- net OUT2-MOTOR-LEFT: now also ARDUINO-MEGA.30
- net OUT2-MOTOR-RIGHT: now also ARDUINO-MEGA.34
- net PWM-MOTOR-LEFT: now also ARDUINO-MEGA.44
- net PWM-MOTOR-RIGHT: now also ARDUINO-MEGA.46
- net SCI: now also ARDUINO-MEGA.47
- net SCL: now also ARDUINO-MEGA.21-SCL
- net SDA: now also ARDUINO-MEGA.20-SDA
- net SERVO1: now also ARDUINO-MEGA.37
- net SERVO2: now also ARDUINO-MEGA.39
- net SERVO3: now also ARDUINO-MEGA.41
- net SERVO4: now also ARDUINO-MEGA.43
- net SHARP-LEFT: now also ARDUINO-MEGA.A5
- net SHARP-MIDDLE: now also ARDUINO-MEGA.A6
- net SHARP-RIGHT: now also ARDUINO-MEGA.A7

Commit message: Preruteo
Parts:
- removed Q1: FDD4141TO252, transistor-fet:FDD4141TO252
- added Q2: TIP41C, transistor-power:TIP41C
- added R-LP: (no value), rcl:R-US_M1206
Connections:
- removed net DRAIN: Q1.D
- removed net GATE: Q1.G
- removed net N$10: ARDUINO-MEGA.49
- removed net N$11: ARDUINO-MEGA.51
- removed net N$12: ARDUINO-MEGA.53
- removed net N$33: ARDUINO-MEGA.50
- removed net N$42: ARDUINO-MEGA.48
- removed net N$43: ARDUINO-MEGA.52
- removed net SOURCE: Q1.S
- new net IOREF: ARDUINO-MEGA.IOREF, U$14.IOREF
- new net N$1: LED_1W.C, Q2.C
- new net N$2: Q2.B, R-LP.2
- new net NC: ARDUINO-MEGA.NC, U$14.NO
- net A10: now also U$9.E7; no longer U$9.E4
- net A11: now also U$9.E9; no longer U$9.E5
- net A12: now also U$9.E11; no longer U$9.E6
- net A13: now also U$9.E13; no longer U$9.E7
- net A14: now also U$9.E12; no longer U$9.E8
- net A15: now also U$9.E10; no longer U$9.E9
- net A9: now also U$9.E5; no longer U$9.E3
- net D36: now also U$9.E2; no longer U$9.E10
- net D38: now also U$9.E4; no longer U$9.E11
- net D40: now also U$9.E6; no longer U$9.E12
- net D42: now also U$9.E8; no longer U$9.E13
- net DIP2: no longer ARDUINO-MEGA.5V_3
- net GND: now also Q2.E
- net LED1W: now also R-LP.1
- net SCD: now also ARDUINO-MEGA.50
- net SF: now also ARDUINO-MEGA.48
- net SID: now also ARDUINO-MEGA.53
- net SII: now also ARDUINO-MEGA.51
- net SSD: now also ARDUINO-MEGA.52
- net SSI: now also ARDUINO-MEGA.49
- net TX2: now also U$9.E3; no longer U$9.E2
- net VCC: now also LED_1W.A
Other:
- moved on the sheet: LED_1W, LINE-SENSOR
