File: Shield/Shield/Shield-Proteco.sch (EAGLE design)
At the start: 53 parts, among them Q2 TIP41C

Commit message: Ruteo
Connections:
- removed net N$38: U$14.NC_1
- net GND: no longer 5V-SOURCE.GND, MOTORS-SOURCE.GND
- net PUSH: no longer PUSH.P1
- net RESET: no longer PUSH-RST.P
- net SCL: no longer ARDUINO-MEGA.SCL
- net SDA: no longer ARDUINO-MEGA.SDA
- net SHARP-LEFT: now also U$14.NC_1
Changed lines of the file:
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@@
 </segment>
 <segment>
-<wire x1="-242.57" y1="171.45" x2="-242.57" y2="168.91" width="0.1524" layer="91"/>
-<wire x1="-242.57" y1="168.91" x2="-238.76" y2="168.91" width="0.1524" layer="91"/>
+<pinref part="GND7" gate="1" pin="GND"/>
+<pinref part="5V-SOURCE" gate="G$1" pin="GND_1"/>
 <wire x1="-238.76" y1="168.91" x2="-234.95" y2="168.91" width="0.1524" layer="91"/>
 <wire x1="-234.95" y1="168.91" x2="-234.95" y2="171.45" width="0.1524" layer="91"/>
-<pinref part="GND7" gate="1" pin="GND"/>
-<junction x="-238.76" y="168.91"/>
-<pinref part="5V-SOURCE" gate="G$1" pin="GND"/>
-<pinref part="5V-SOURCE" gate="G$1" pin="GND_1"/>
 </segment>
 <segment>
@@
 <segment>
 <pinref part="GND12" gate="1" pin="GND"/>
-<wire x1="-242.57" y1="137.16" x2="-242.57" y2="132.08" width="0.1524" layer="91"/>
-<wire x1="-242.57" y1="132.08" x2="-238.76" y2="132.08" width="0.1524" layer="91"/>
 <wire x1="-238.76" y1="132.08" x2="-234.95" y2="132.08" width="0.1524" layer="91"/>
 <wire x1="-234.95" y1="132.08" x2="-234.95" y2="137.16" width="0.1524" layer="91"/>
-<junction x="-238.76" y="132.08"/>
-<pinref part="MOTORS-SOURCE" gate="G$1" pin="GND"/>
 <pinref part="MOTORS-SOURCE" gate="G$1" pin="GND_1"/>
 </segment>
@@
 <label x="24.13" y="-38.1" size="1.778" layer="95" rot="R180" xref="yes"/>
 </segment>
+<segment>
+<pinref part="U$14" gate="G$1" pin="NC_1"/>
+<wire x1="284.48" y1="-2.54" x2="278.13" y2="-2.54" width="0.1524" layer="91"/>
+<label x="278.13" y="-2.54" size="1.778" layer="95" rot="R180" xref="yes"/>
+</segment>
 </net>
 <net name="SHARP-MIDDLE" class="0">
@@
 <net name="PUSH" class="0">
 <segment>
-<pinref part="PUSH" gate="1" pin="P"/>
-<pinref part="RPUSH-2" gate="G$1" pin="2"/>
-<wire x1="-138.43" y1="127" x2="-135.89" y2="128.27" width="0.1524" layer="91"/>
-<junction x="-138.43" y="127"/>
-<label x="-132.08" y="128.27" size="1.778" layer="95" xref="yes"/>
-<pinref part="PUSH" gate="1" pin="P1"/>
-<wire x1="-135.89" y1="128.27" x2="-132.08" y2="128.27" width="0.1524" layer="91"/>
-<junction x="-135.89" y="128.27"/>
-<wire x1="-138.43" y1="127" x2="-138.43" y2="128.27" width="0.1524" layer="91"/>
-</segment>
-<segment>
 <pinref part="ARDUINO-MEGA" gate="G$1" pin="25"/>
 <wire x1="95.25" y1="-106.68" x2="95.25" y2="-124.46" width="0.1524" layer="91"/>
 <label x="95.25" y="-124.46" size="1.778" layer="95" rot="R270" xref="yes"/>
+</segment>
+<segment>
+<pinref part="PUSH" gate="1" pin="P"/>
+<pinref part="RPUSH-2" gate="G$1" pin="2"/>
+<wire x1="-138.43" y1="128.27" x2="-138.43" y2="127" width="0.1524" layer="91"/>
+<wire x1="-138.43" y1="127" x2="-133.35" y2="127" width="0.1524" layer="91"/>
+<junction x="-138.43" y="127"/>
+<label x="-133.35" y="127" size="1.778" layer="95" xref="yes"/>
 </segment>
 </net>
@@
 </segment>
 <segment>
-<pinref part="PUSH-RST" gate="1" pin="P"/>
-<wire x1="-165.1" y1="128.27" x2="-162.56" y2="128.27" width="0.1524" layer="91"/>
 <label x="-158.75" y="128.27" size="1.778" layer="95" xref="yes"/>
 <pinref part="PUSH-RST" gate="1" pin="P1"/>
 <wire x1="-162.56" y1="128.27" x2="-158.75" y2="128.27" width="0.1524" layer="91"/>
-<junction x="-162.56" y="128.27"/>
 </segment>
 </net>
@@
 </segment>
 <segment>
-<pinref part="ARDUINO-MEGA" gate="G$1" pin="SCL"/>
-<wire x1="110.49" y1="2.54" x2="118.11" y2="2.54" width="0.1524" layer="91"/>
-<label x="118.11" y="2.54" size="1.778" layer="95" xref="yes"/>
-</segment>
-<segment>
 <pinref part="ARDUINO-MEGA" gate="G$1" pin="21-SCL"/>
 <wire x1="110.49" y1="-68.58" x2="127" y2="-68.58" width="0.1524" layer="91"/>
@@
 </segment>
 <segment>
-<pinref part="ARDUINO-MEGA" gate="G$1" pin="SDA"/>
-<wire x1="110.49" y1="0" x2="127" y2="0" width="0.1524" layer="91"/>
-<label x="127" y="0" size="1.778" layer="95" xref="yes"/>
-</segment>
-<segment>
 <pinref part="ARDUINO-MEGA" gate="G$1" pin="20-SDA"/>
 <wire x1="110.49" y1="-66.04" x2="114.3" y2="-66.04" width="0.1524" layer="91"/>
@@
 </segment>
 </net>
-<net name="N$38" class="0">
-<segment>
-<pinref part="U$14" gate="G$1" pin="NC_1"/>
-<wire x1="284.48" y1="-2.54" x2="278.13" y2="-2.54" width="0.1524" layer="91"/>
-<label x="278.13" y="-2.54" size="1.778" layer="95" rot="R180" xref="yes"/>
-</segment>
-</net>

Commit message: Ruteo avance
Connections:
- net IN1-MOTOR-LEFT: now also ARDUINO-MEGA.30
- net IN1-MOTOR-RIGHT: now also ARDUINO-MEGA.32
- net IN2-MOTOR-LEFT: now also ARDUINO-MEGA.28
- net IN2-MOTOR-RIGHT: now also ARDUINO-MEGA.34
- net OUT1-MOTOR-LEFT: no longer ARDUINO-MEGA.28
- net OUT1-MOTOR-RIGHT: no longer ARDUINO-MEGA.32
- net OUT2-MOTOR-LEFT: no longer ARDUINO-MEGA.30
- net OUT2-MOTOR-RIGHT: no longer ARDUINO-MEGA.34
Changed lines of the file:
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@@
 <label x="-232.41" y="-1.27" size="1.778" layer="95" xref="yes"/>
+</segment>
+<segment>
+<pinref part="ARDUINO-MEGA" gate="G$1" pin="30"/>
+<wire x1="87.63" y1="-83.82" x2="87.63" y2="-54.61" width="0.1524" layer="91"/>
+<label x="87.63" y="-54.61" size="1.778" layer="95" rot="R90" xref="yes"/>
 </segment>
 </net>
@@
 <junction x="-241.3" y="-10.16"/>
 <label x="-227.33" y="-10.16" size="1.778" layer="95" xref="yes"/>
+</segment>
+<segment>
+<pinref part="ARDUINO-MEGA" gate="G$1" pin="28"/>
+<wire x1="90.17" y1="-83.82" x2="90.17" y2="-82.55" width="0.1524" layer="91"/>
+<label x="90.17" y="-82.55" size="1.778" layer="95" rot="R90" xref="yes"/>
 </segment>
 </net>
@@
 <label x="-97.79" y="3.81" size="1.778" layer="95" xref="yes"/>
 </segment>
-<segment>
-<pinref part="ARDUINO-MEGA" gate="G$1" pin="30"/>
-<wire x1="87.63" y1="-83.82" x2="87.63" y2="-54.61" width="0.1524" layer="91"/>
-<label x="87.63" y="-54.61" size="1.778" layer="95" rot="R90" xref="yes"/>
-</segment>
 </net>
 <net name="OUT1-MOTOR-LEFT" class="0">
@@
 <wire x1="-111.76" y1="6.35" x2="-106.68" y2="6.35" width="0.1524" layer="91"/>
 <label x="-106.68" y="6.35" size="1.778" layer="95" xref="yes"/>
-</segment>
-<segment>
-<pinref part="ARDUINO-MEGA" gate="G$1" pin="28"/>
-<wire x1="90.17" y1="-83.82" x2="90.17" y2="-82.55" width="0.1524" layer="91"/>
-<label x="90.17" y="-82.55" size="1.778" layer="95" rot="R90" xref="yes"/>
 </segment>
 </net>
@@
 <label x="-232.41" y="-53.34" size="1.778" layer="95" xref="yes"/>
 </segment>
+<segment>
+<pinref part="ARDUINO-MEGA" gate="G$1" pin="34"/>
+<wire x1="82.55" y1="-83.82" x2="82.55" y2="-54.61" width="0.1524" layer="91"/>
+<label x="82.55" y="-54.61" size="1.778" layer="95" rot="R90" xref="yes"/>
+</segment>
 </net>
 <net name="IN1-MOTOR-RIGHT" class="0">
@@
 <junction x="-243.84" y="-46.99"/>
 <label x="-231.14" y="-46.99" size="1.778" layer="95" xref="yes"/>
+</segment>
+<segment>
+<pinref part="ARDUINO-MEGA" gate="G$1" pin="32"/>
+<wire x1="85.09" y1="-83.82" x2="85.09" y2="-82.55" width="0.1524" layer="91"/>
+<label x="85.09" y="-82.55" size="1.778" layer="95" rot="R90" xref="yes"/>
 </segment>
 </net>
@@
 <label x="-83.82" y="-31.75" size="1.778" layer="95" xref="yes"/>
 </segment>
-<segment>
-<pinref part="ARDUINO-MEGA" gate="G$1" pin="34"/>
-<wire x1="82.55" y1="-83.82" x2="82.55" y2="-54.61" width="0.1524" layer="91"/>
-<label x="82.55" y="-54.61" size="1.778" layer="95" rot="R90" xref="yes"/>
-</segment>
 </net>
 <net name="OUT1-MOTOR-RIGHT" class="0">
@@
 <label x="-105.41" y="-29.21" size="1.778" layer="95" xref="yes"/>
 </segment>
-<segment>
-<pinref part="ARDUINO-MEGA" gate="G$1" pin="32"/>
-<wire x1="85.09" y1="-83.82" x2="85.09" y2="-82.55" width="0.1524" layer="91"/>
-<label x="85.09" y="-82.55" size="1.778" layer="95" rot="R90" xref="yes"/>
-</segment>
 </net>

Commit message: Ruote Finish
Connections:
- net DIP3: now also ARDUINO-MEGA.26; no longer ARDUINO-MEGA.24
- net DIP4: now also ARDUINO-MEGA.24; no longer ARDUINO-MEGA.26
Changed lines of the file:
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@@
 </segment>
 <segment>
-<pinref part="ARDUINO-MEGA" gate="G$1" pin="24"/>
-<wire x1="95.25" y1="-83.82" x2="95.25" y2="-82.55" width="0.1524" layer="91"/>
-<label x="95.25" y="-82.55" size="1.778" layer="95" rot="R90" xref="yes"/>
+<pinref part="ARDUINO-MEGA" gate="G$1" pin="26"/>
+<wire x1="92.71" y1="-83.82" x2="92.71" y2="-72.39" width="0.1524" layer="91"/>
+<label x="92.71" y="-72.39" size="1.778" layer="95" rot="R90" xref="yes"/>
 </segment>
 </net>
@@
 </segment>
 <segment>
-<pinref part="ARDUINO-MEGA" gate="G$1" pin="26"/>
-<wire x1="92.71" y1="-83.82" x2="92.71" y2="-72.39" width="0.1524" layer="91"/>
-<label x="92.71" y="-72.39" size="1.778" layer="95" rot="R90" xref="yes"/>
+<pinref part="ARDUINO-MEGA" gate="G$1" pin="24"/>
+<wire x1="95.25" y1="-83.82" x2="95.25" y2="-82.55" width="0.1524" layer="91"/>
+<label x="95.25" y="-82.55" size="1.778" layer="95" rot="R90" xref="yes"/>
 </segment>
 </net>

Commit message: Ruteo Ajustes
Connections:
- net VCC: now also DRIVER-LEFT.STBY, DRIVER-RIGHT.STBY
Changed lines of the file:
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@@
 <part name="P+10" library="supply1" library_urn="urn:adsk.eagle:library:371" deviceset="VCC" device=""/>
 <part name="GND8" library="supply1" library_urn="urn:adsk.eagle:library:371" deviceset="GND" device=""/>
+<part name="P+11" library="supply1" library_urn="urn:adsk.eagle:library:371" deviceset="VCC" device=""/>
 </parts>
 <sheets>
@@
 <instance part="P+10" gate="VCC" x="220.98" y="-160.02"/>
 <instance part="GND8" gate="1" x="220.98" y="-198.12"/>
+<instance part="P+11" gate="VCC" x="-246.38" y="-20.32"/>
 </instances>
 <busses>
@@
 <wire x1="220.98" y1="-162.56" x2="220.98" y2="-167.64" width="0.1524" layer="91"/>
 </segment>
+<segment>
+<pinref part="DRIVER-LEFT" gate="G$1" pin="STBY"/>
+<wire x1="-257.81" y1="0" x2="-252.73" y2="0" width="0.1524" layer="91"/>
+<wire x1="-252.73" y1="0" x2="-252.73" y2="-27.94" width="0.1524" layer="91"/>
+<pinref part="DRIVER-RIGHT" gate="G$1" pin="STBY"/>
+<wire x1="-252.73" y1="-27.94" x2="-252.73" y2="-53.34" width="0.1524" layer="91"/>
+<wire x1="-252.73" y1="-53.34" x2="-257.81" y2="-53.34" width="0.1524" layer="91"/>
+<pinref part="P+11" gate="VCC" pin="VCC"/>
+<wire x1="-252.73" y1="-27.94" x2="-246.38" y2="-27.94" width="0.1524" layer="91"/>
+<wire x1="-246.38" y1="-27.94" x2="-246.38" y2="-22.86" width="0.1524" layer="91"/>
+<junction x="-252.73" y="-27.94"/>
+</segment>
 </net>

Commit message: Retoques
Parts:
- added U$1: LIPO7.4MOLEX, Baterias:LIPO7.4MOLEX
Connections:
- removed net N$14: 5V-SOURCE.VIN, MOTORS-SOURCE.VIN, POWER-SW.2
- net GND: now also U$1.GND
- net N$134: now also U$1.7.4V
- net VIN: now also 5V-SOURCE.VIN, MOTORS-SOURCE.VIN, POWER-SW.2

Commit message: Shield Terminada
Parts:
- added C1: (no value), rcl:CPOL-USE5-10.5
Connections:
- net GND: now also C1.-
- net VCC: now also C1.+
